File: hardware/board-stm32-v1/actuator-v1/MCU-STM32G0B1RBT6.kicad_sch (KiCad schematic)
At the start: 19 parts, among them SW1 SW_Push, U2 STM32G0B1CBT6, X1 32.768KHz, X2 8MHz

Commit message: Update actuator PCB layout and schematics
Connections:
- net ADC1_IN0: now also U2.12 (PA1); no longer U2.11 (PA0)
- net ADC1_IN1: now also U2.11 (PA0); no longer U2.12 (PA1)
Changed lines of the file:
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@@
 		)
 	)
-	(hierarchical_label "ADC1_IN0"
+	(hierarchical_label "ADC1_IN1"
 		(shape bidirectional)
 		(at 137.16 44.45 0)
@@
 		)
 	)
-	(hierarchical_label "ADC1_IN1"
+	(hierarchical_label "ADC1_IN0"
 		(shape bidirectional)
 		(at 137.16 46.99 0)
