File: hardware/board-stm32-v1/actuator-v1/TCAN3413.kicad_sch (KiCad schematic)
At the start: 14 parts, among them IC1 TCAN3413DR, J2 Screw_Terminal_01x03

Commit message: Update actuator PCB layout and schematics
Connections:
- net CAN+: no longer IC1.7 (CANH), L1.1
- net CAN-: no longer IC1.6 (CANL), L1.2
- new net: IC1.7 (CANH), L1.1
- new net: IC1.6 (CANL), L1.2
Changed lines of the file:
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@@
-		)
-	)
-	(label "CAN+"
-		(at 109.22 69.85 0)
-		(fields_autoplaced yes)
-		(effects
-			(font
-				(size 1.27 1.27)
-			)
-			(justify left bottom)
-		)
-		(property "Net Class" "CAN"
-			(at 109.22 71.12 0)
-			(show_name no)
-			(do_not_autoplace no)
-			(effects
-				(font
-					(size 1.27 1.27)
-					(italic yes)
-				)
-				(justify left)
-			)
 		)
 	)
@@
 			(show_name no)
 			(do_not_autoplace no)
-			(effects
-				(font
-					(size 1.27 1.27)
-					(italic yes)
-				)
-				(justify left)
-			)
-		)
-	)
-	(label "CAN-"
-		(at 109.22 82.55 0)
-		(fields_autoplaced yes)
-		(effects
-			(font
-				(size 1.27 1.27)
-			)
-			(justify left bottom)
-		)
-		(property "Net Class" "CAN"
-			(at 109.22 83.82 0)
-			(show_name no)
-			(do_not_autoplace no)
